File: simo-botella.kicad_pcb (KiCad board)
At the start: 2 copper layers, 1 part

Commit message: update
Parts:
- moved REF** 130.2 mm to (122.0, 195.0)
Other:
- board outline added: 200 x 70 mm
Changed lines of the file:
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@@
   (net 0 "")
   (footprint "simo-shield:simo-shield" (layer "F.Cu")
-    (at 130 65)
+    (at 122 195)
     (attr through_hole)
     (fp_text reference "REF**" (at -50 -35.5 unlocked) (layer "F.SilkS")
@@
     (pad "1" thru_hole circle (at -43 27) (size 1.5 1.5) (drill 1) (layers *.Cu *.Mask "Dwgs.User"))
   )
-  (gr_line (start 45 30) (end 45 100) (layer "Dwgs.User") (width 0.15))
-  (gr_rect (start 45 30) (end 80 100) (layer "Dwgs.User") (width 0.15) (fill none))
-  (gr_line (start 185 90) (end 245 90) (layer "Dwgs.User") (width 0.15))
-  (gr_line (start 245 90) (end 245 30) (layer "Dwgs.User") (width 0.15))
-  (gr_line (start 185 100) (end 45 100) (layer "Dwgs.User") (width 0.15))
-  (gr_line (start 185 90) (end 185 100) (layer "Dwgs.User") (width 0.15))
-  (gr_line (start 245 30) (end 45 30) (layer "Dwgs.User") (width 0.15))
+  (gr_rect (start 14 160) (end 49 230) (layer "Dwgs.User") (width 0.15) (fill none))
+  (gr_line (start 45 30) (end 45 100) (layer "Edge.Cuts") (width 0.15))
+  (gr_line (start 185 90) (end 245 90) (layer "Edge.Cuts") (width 0.15))
+  (gr_line (start 245 90) (end 245 30) (layer "Edge.Cuts") (width 0.15))
+  (gr_line (start 185 100) (end 45 100) (layer "Edge.Cuts") (width 0.15))
+  (gr_line (start 185 90) (end 185 100) (layer "Edge.Cuts") (width 0.15))
+  (gr_line (start 245 30) (end 45 30) (layer "Edge.Cuts") (width 0.15))
   (gr_text "Tenemos: Simo-shield medida 70 mm x 100 mm. \n4 Agujeros (separacion54 mm x 86mm )\nPlaca switch magnetico: 35mm x 7mm \nagujeros alineados con simo-shield.\nMe falta dato de curvatura para elegir un diametro de cilindro." (at 34 134) (layer "Dwgs.User")
     (effects (font (size 1.2 1.2) (thickness 0.15)) (justify left))
@@
   )
   (dimension (type aligned) (layer "Dwgs.User")
-    (pts (xy 245 30) (xy 245 90))
+    (pts (xy 256 30) (xy 256 90))
     (height -15)
-    (gr_text "60,0000 mm" (at 258.85 60 90) (layer "Dwgs.User")
+    (gr_text "60,0000 mm" (at 269.85 60 90) (layer "Dwgs.User")
       (effects (font (size 1 1) (thickness 0.15)))
     )
@@
   )
   (dimension (type aligned) (layer "Dwgs.User")
-    (pts (xy 40 30) (xy 40 100))
+    (pts (xy 39 30) (xy 39 100))
     (height 23)
-    (gr_text "70,0000 mm" (at 15.85 65 90) (layer "Dwgs.User")
+    (gr_text "70,0000 mm" (at 14.85 65 90) (layer "Dwgs.User")
       (effects (font (size 1 1) (thickness 0.15)))
     )
